File: eagle/damper-controller/v1.sch (EAGLE design)
At the start: 18 parts, among them IC1 ULN2003AD, Q1 RS485-ADAPTER0.05-CONNECTOR

Commit message: Finished damper controller, and modified for OSH Park print, instead of home-made method
Parts:
- removed LED1, LED2, LED3, LED4: (no value), led:LEDSML1206
- removed R1, R2, R3, R4: 2k2, resistor:R-US_R0603
- R5: value 1k -> 10k
Connections:
- removed net N$6: LED4.A, R4.1
- removed net N$7: LED3.A, R3.1
- removed net N$8: LED2.A, R2.1
- removed net N$9: LED1.A, R1.1
- net GND: no longer LED1.C, LED2.C, LED3.C, LED4.C
- net N$2: no longer R1.2
- net N$3: no longer R2.2
- net N$4: no longer R3.2
- net N$5: no longer R4.2
Changed lines of the file:
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@@
 <part name="ENDSTOP" library="con-amp-quick" deviceset="M02" device=""/>
 <part name="C1" library="eagle-ltspice" deviceset="C" device="C0603"/>
-<part name="LED1" library="led" deviceset="LED" device="SML1206"/>
-<part name="LED2" library="led" deviceset="LED" device="SML1206"/>
-<part name="LED3" library="led" deviceset="LED" device="SML1206"/>
-<part name="LED4" library="led" deviceset="LED" device="SML1206"/>
-<part name="R1" library="resistor" deviceset="R-US_" device="R0603" value="2k2"/>
-<part name="R2" library="resistor" deviceset="R-US_" device="R0603" value="2k2"/>
-<part name="R3" library="resistor" deviceset="R-US_" device="R0603" value="2k2"/>
-<part name="R4" library="resistor" deviceset="R-US_" device="R0603" value="2k2"/>
 <part name="P+3" library="supply1" deviceset="+12V" device=""/>
-<part name="GND2" library="supply1" deviceset="GND" device=""/>
 <part name="GND3" library="supply1" deviceset="GND" device=""/>
 <part name="P+2" library="supply1" deviceset="+12V" device=""/>
@@
 <part name="GND5" library="supply1" deviceset="GND" device=""/>
 <part name="LED5" library="led" deviceset="LED" device="SML1206"/>
-<part name="R5" library="resistor" deviceset="R-US_" device="R0603" value="1k"/>
+<part name="R5" library="resistor" deviceset="R-US_" device="R0603" value="10k"/>
 <part name="P+6" library="supply1" deviceset="VCC" device=""/>
 <part name="I2C" library="con-amp-quick" deviceset="M04" device=""/>
@@
 <instance part="ENDSTOP" gate="G$1" x="88.9" y="116.84" rot="R180"/>
 <instance part="C1" gate="G$1" x="38.1" y="25.4" rot="R270"/>
-<instance part="LED1" gate="G$1" x="96.52" y="60.96" rot="R90"/>
-<instance part="LED2" gate="G$1" x="96.52" y="53.34" rot="R90"/>
-<instance part="LED3" gate="G$1" x="96.52" y="45.72" rot="R90"/>
-<instance part="LED4" gate="G$1" x="96.52" y="38.1" rot="R90"/>
-<instance part="R1" gate="G$1" x="86.36" y="60.96" rot="R180"/>
-<instance part="R2" gate="G$1" x="86.36" y="53.34" rot="R180"/>
-<instance part="R3" gate="G$1" x="86.36" y="45.72" rot="R180"/>
-<instance part="R4" gate="G$1" x="86.36" y="38.1" rot="R180"/>
 <instance part="P+3" gate="1" x="58.42" y="38.1" rot="R270"/>
-<instance part="GND2" gate="1" x="106.68" y="27.94"/>
 <instance part="GND3" gate="1" x="22.86" y="20.32"/>
 <instance part="P+2" gate="1" x="10.16" y="86.36" rot="R90"/>
@@
 <wire x1="50.8" y1="55.88" x2="73.66" y2="55.88" width="0.1524" layer="91"/>
 <wire x1="73.66" y1="55.88" x2="73.66" y2="30.48" width="0.1524" layer="91"/>
-<pinref part="R1" gate="G$1" pin="2"/>
-<wire x1="81.28" y1="60.96" x2="73.66" y2="60.96" width="0.1524" layer="91"/>
-<wire x1="73.66" y1="60.96" x2="73.66" y2="55.88" width="0.1524" layer="91"/>
-<junction x="73.66" y="55.88"/>
 </segment>
 </net>
@@
 <segment>
 <pinref part="MOTOR" gate="G$1" pin="2"/>
-<wire x1="71.12" y1="53.34" x2="71.12" y2="50.8" width="0.1524" layer="91"/>
-<pinref part="R2" gate="G$1" pin="2"/>
 <wire x1="71.12" y1="50.8" x2="71.12" y2="30.48" width="0.1524" layer="91"/>
-<wire x1="81.28" y1="53.34" x2="71.12" y2="53.34" width="0.1524" layer="91"/>
 <pinref part="IC1" gate="A" pin="O3"/>
 <wire x1="50.8" y1="50.8" x2="71.12" y2="50.8" width="0.1524" layer="91"/>
-<junction x="71.12" y="50.8"/>
 </segment>
 </net>
@@
 <segment>
 <pinref part="MOTOR" gate="G$1" pin="3"/>
-<pinref part="R3" gate="G$1" pin="2"/>
 <wire x1="68.58" y1="45.72" x2="68.58" y2="30.48" width="0.1524" layer="91"/>
-<wire x1="81.28" y1="45.72" x2="68.58" y2="45.72" width="0.1524" layer="91"/>
-<junction x="68.58" y="45.72"/>
 <pinref part="IC1" gate="A" pin="O5"/>
 <wire x1="50.8" y1="45.72" x2="68.58" y2="45.72" width="0.1524" layer="91"/>
@@
 <segment>
 <pinref part="MOTOR" gate="G$1" pin="4"/>
-<pinref part="R4" gate="G$1" pin="2"/>
-<wire x1="66.04" y1="40.64" x2="66.04" y2="38.1" width="0.1524" layer="91"/>
-<wire x1="66.04" y1="38.1" x2="66.04" y2="30.48" width="0.1524" layer="91"/>
-<wire x1="81.28" y1="38.1" x2="66.04" y2="38.1" width="0.1524" layer="91"/>
-<junction x="66.04" y="38.1"/>
+<wire x1="66.04" y1="40.64" x2="66.04" y2="30.48" width="0.1524" layer="91"/>
 <pinref part="IC1" gate="A" pin="O7"/>
 <wire x1="50.8" y1="40.64" x2="66.04" y2="40.64" width="0.1524" layer="91"/>
 </segment>
 </net>
-<net name="N$6" class="0">
-<segment>
-<pinref part="R4" gate="G$1" pin="1"/>
-<pinref part="LED4" gate="G$1" pin="A"/>
-<wire x1="91.44" y1="38.1" x2="93.98" y2="38.1" width="0.1524" layer="91"/>
-</segment>
-</net>
-<net name="N$7" class="0">
-<segment>
-<pinref part="LED3" gate="G$1" pin="A"/>
-<pinref part="R3" gate="G$1" pin="1"/>
-<wire x1="93.98" y1="45.72" x2="91.44" y2="45.72" width="0.1524" layer="91"/>
-</segment>
-</net>
-<net name="N$8" class="0">
-<segment>
-<pinref part="R2" gate="G$1" pin="1"/>
-<pinref part="LED2" gate="G$1" pin="A"/>
-<wire x1="91.44" y1="53.34" x2="93.98" y2="53.34" width="0.1524" layer="91"/>
-</segment>
-</net>
-<net name="N$9" class="0">
-<segment>
-<pinref part="LED1" gate="G$1" pin="A"/>
-<pinref part="R1" gate="G$1" pin="1"/>
-<wire x1="93.98" y1="60.96" x2="91.44" y2="60.96" width="0.1524" layer="91"/>
-</segment>
-</net>
 <net name="GND" class="0">
 <segment>
-<pinref part="LED1" gate="G$1" pin="C"/>
-<pinref part="GND2" gate="1" pin="GND"/>
-<wire x1="101.6" y1="60.96" x2="106.68" y2="60.96" width="0.1524" layer="91"/>
-<wire x1="106.68" y1="60.96" x2="106.68" y2="53.34" width="0.1524" layer="91"/>
-<pinref part="LED4" gate="G$1" pin="C"/>
-<wire x1="106.68" y1="53.34" x2="106.68" y2="45.72" width="0.1524" layer="91"/>
-<wire x1="106.68" y1="45.72" x2="106.68" y2="38.1" width="0.1524" layer="91"/>
-<wire x1="106.68" y1="38.1" x2="106.68" y2="30.48" width="0.1524" layer="91"/>
-<wire x1="101.6" y1="38.1" x2="106.68" y2="38.1" width="0.1524" layer="91"/>
-<junction x="106.68" y="38.1"/>
-<pinref part="LED3" gate="G$1" pin="C"/>
-<wire x1="101.6" y1="45.72" x2="106.68" y2="45.72" width="0.1524" layer="91"/>
-<junction x="106.68" y="45.72"/>
-<pinref part="LED2" gate="G$1" pin="C"/>
-<wire x1="101.6" y1="53.34" x2="106.68" y2="53.34" width="0.1524" layer="91"/>
-<junction x="106.68" y="53.34"/>
-</segment>
-<segment>
 <pinref part="C1" gate="G$1" pin="2"/>

Commit message: Adjusting damper controller board based on first prototype of PCB. Needed to move switch connector, and removed LED, as there is no space.
Parts:
- removed LED5: (no value), led:LEDSML1206
- removed R5: 10k, resistor:R-US_R0603
Connections:
- removed net N$13: LED5.A, R5.2
- net N$12: no longer LED5.C
- net VCC: no longer R5.1
Changed lines of the file:
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@@
 <part name="P+5" library="supply1" deviceset="VCC" device=""/>
 <part name="GND5" library="supply1" deviceset="GND" device=""/>
-<part name="LED5" library="led" deviceset="LED" device="SML1206"/>
-<part name="R5" library="resistor" deviceset="R-US_" device="R0603" value="10k"/>
-<part name="P+6" library="supply1" deviceset="VCC" device=""/>
 <part name="I2C" library="con-amp-quick" deviceset="M04" device=""/>
 <part name="P+7" library="supply1" deviceset="VCC" device=""/>
@@
 <instance part="P+5" gate="VCC" x="10.16" y="78.74" rot="R90"/>
 <instance part="GND5" gate="1" x="78.74" y="106.68"/>
-<instance part="LED5" gate="G$1" x="83.82" y="124.46" rot="R270"/>
-<instance part="R5" gate="G$1" x="93.98" y="124.46" rot="R180"/>
-<instance part="P+6" gate="VCC" x="106.68" y="124.46" rot="R270"/>
 <instance part="I2C" gate="G$1" x="93.98" y="147.32" rot="R180"/>
 <instance part="P+7" gate="VCC" x="83.82" y="157.48"/>
@@
 </segment>
 <segment>
-<pinref part="P+6" gate="VCC" pin="VCC"/>
-<pinref part="R5" gate="G$1" pin="1"/>
-<wire x1="104.14" y1="124.46" x2="99.06" y2="124.46" width="0.1524" layer="91"/>
-</segment>
-<segment>
 <pinref part="I2C" gate="G$1" pin="1"/>
 <pinref part="P+7" gate="VCC" pin="VCC"/>
@@
 <pinref part="ENDSTOP" gate="G$1" pin="1"/>
 <pinref part="U$1" gate="G$1" pin="D3"/>
-<wire x1="81.28" y1="116.84" x2="76.2" y2="116.84" width="0.1524" layer="91"/>
-<pinref part="LED5" gate="G$1" pin="C"/>
-<wire x1="76.2" y1="116.84" x2="58.42" y2="116.84" width="0.1524" layer="91"/>
-<wire x1="78.74" y1="124.46" x2="76.2" y2="124.46" width="0.1524" layer="91"/>
-<wire x1="76.2" y1="124.46" x2="76.2" y2="116.84" width="0.1524" layer="91"/>
-<junction x="76.2" y="116.84"/>
-</segment>
-</net>
-<net name="N$13" class="0">
-<segment>
-<pinref part="R5" gate="G$1" pin="2"/>
-<pinref part="LED5" gate="G$1" pin="A"/>
-<wire x1="88.9" y1="124.46" x2="86.36" y2="124.46" width="0.1524" layer="91"/>
-</segment>
-</net>
+<wire x1="81.28" y1="116.84" x2="58.42" y2="116.84" width="0.1524" layer="91"/>
+</segment>
+</net>
