File: eagle/mainboard/mainboard-v2-opto.brd (EAGLE design)
At the start: 100 x 80 mm, 64 parts, among them K1 TQ2-SA-12V, K2 TQ2-SA-12V, K3 TQ2-SA-12V, K4 TQ2-SA-12V, K5 TQ2-SA-12V, K6 TQ2-SA-12V, K7 TQ2-SA-12V, K8 TQ2-SA-12V, Q1 RS485-ADAPTER0.05-CONNECTOR

Commit message: Starting work on solid state relay version of mainboard, as it's much more manageable (albeit still painful)
Parts:
- removed D2, D3, D4, D5, D6: (no value), adafruit:SMADIODE
- removed K4, K5, K6, K7, K8: TQ2-SA-12V, relay:TQ-SA
- removed T2, T3, T4, T5, T6: (no value), transistor:SOT23-BEC
- added K10, K11, K12, K13, K9: AQY21SOP, relay:SOP04
- R12, R13, R14, R15, R16: value 2k2 -> 470
- T1-C, T1-G, T1-R, T1-W1, T1-W2, T1-Y1, T1-Y2, UNIT-C, UNIT-G, UNIT-R, UNIT-W1, UNIT-W2, UNIT-Y1, UNIT-Y2: device wirepad:1,6/0,9 -> wirepad:2,15/1,0
- moved Q1 15.7 mm to (21.6, 45.7)
- moved T1-R 7.62 mm to (5.08, 10.2), turned to 0 degrees
- moved UNIT-R 7.62 mm to (10.2, 5.08)
- moved R10 2.62 mm to (21.0, 41.9)
- moved R6 2.62 mm to (17.1, 41.9)
- moved B4 2.62 mm to (10.8, 30.5)
- moved B5 2.62 mm to (10.8, 25.4)
- moved C1 2.62 mm to (17.1, 24.1)
- moved R8 2.62 mm to (22.2, 31.8)
- moved B1 2.62 mm to (10.8, 20.3)
- moved B2 2.62 mm to (10.8, 40.6)
- moved B3 2.62 mm to (10.8, 35.6)
- moved C2 2.62 mm to (17.1, 29.2)
- moved C3 2.62 mm to (17.1, 34.3)
- moved C4 2.62 mm to (17.1, 39.4)
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Connections:
- removed net N$21: D2.A, K4.10, T2.C
- removed net N$25: D3.A, K5.10, T6.C
- removed net N$26: D5.A, K7.10, T5.C
- removed net N$28: D4.A, K6.10, T3.C
- removed net N$31: D6.A, K8.10, T4.C
- removed net N$33: R12.2, T2.B
- removed net N$36: R15.2, T3.B
- removed net N$38: R14.2, T5.B
- removed net N$40: R16.2, T4.B
- new net N$11: K12.1, R16.2
- new net N$12: K11.1, R15.2
- new net N$16: K9.1, R12.2
- new net N$8: K13.1, R14.2
- net +12V: no longer D2.C, D3.C, D4.C, D5.C, D6.C, K4.1, K5.1, K6.1, K7.1, K8.1
- net 24VAC-R: now also K10.3, K11.3, K12.3, K13.3, K9.3; no longer K4.8, K5.8, K6.8, K7.8, K8.8
- net GND: now also K10.2, K11.2, K12.2, K13.2, K9.2; no longer T2.E, T3.E, T4.E, T5.E, T6.E
- net N$32: no longer T6.B
- net N$4: now also K2.8; no longer K2.3
- net N$7: now also K2.3; no longer K2.8
- net PI-G: now also K9.4; no longer K8.7
- net PI-W1: now also K12.4, K2.7; no longer K2.4, K4.7
- net PI-W2: now also K13.4; no longer K5.7
- net PI-Y1: now also K10.4; no longer K6.7
- net PI-Y2: now also K11.4, K2.4; no longer K2.7, K7.7
- net T1-W1: now also K2.2; no longer K2.9
- net T1-Y2: now also K2.9; no longer K2.2
Routing:
- net +12V: track 0.00 -> 79.9 mm, vias 0 -> 4
- net 24VAC-R: track 18.0 -> 90.4 mm
- net N$5: track 0.00 -> 53.5 mm, vias 0 -> 2
- net PI-Y2: track 0.00 -> 20.8 mm, vias 0 -> 1
- net PI-W1: track 0.00 -> 19.0 mm, vias 0 -> 1
- net RX: track 0.00 -> 17.1 mm
- net TX: track 0.00 -> 14.8 mm
- net +5V: track 0.00 -> 13.0 mm
- net N$24: track 28.0 -> 15.6 mm
- net PI-W2: track 0.00 -> 12.2 mm, vias 0 -> 1
- net PI-G: track 0.00 -> 10.7 mm, vias 0 -> 1
- net N$23: track 28.6 -> 18.5 mm
- net N$19: track 40.2 -> 30.1 mm
- net 4: track 0.00 -> 9.94 mm
- net PI-Y1: track 0.00 -> 7.88 mm, vias 0 -> 1
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
Commit message: Really close to finishing first prototype of the motherboard.
Parts:
- removed SL1: (no value), con-amp-quick:04P
- added I2C, RS1: (no value), con-amp-quick:04P
- added U$2: SWITCH-1, serge:SWITCH-1
- moved R1 127.8 mm to (43.2, 33.0), flipped to the bottom, turned to 270 degrees
- moved R13 124.0 mm to (48.3, 11.4), flipped to the bottom
- moved T1 118.7 mm to (41.9, 28.6), flipped to the bottom, turned to 270 degrees
- moved R16 117.5 mm to (36.8, 32.4), flipped to the bottom
- moved R12 109.2 mm to (33.7, 9.53), flipped to the bottom, turned to 90 degrees
- moved R14 108.8 mm to (32.4, 22.9), flipped to the bottom, turned to 270 degrees
- moved D1 102.5 mm to (50.8, 24.8), flipped to the bottom
- moved R15 101.5 mm to (28.6, 41.9), flipped to the bottom, turned to 270 degrees
- moved Q1 0.90 mm to (22.2, 46.4)
Connections:
- removed net 24: R11.1, R7.2
- removed net N$19: CN1.PWR, Q1.12V-IN, SL1.1
- removed net N$23: Q1.A, SL1.2
- removed net N$24: Q1.B, SL1.3
- removed net N$32: R13.2
- new net 25: R14.1, U$1.P$22
- new net 27: R4.2, R8.1, U$1.P$13
- new net N$17: K10.1, R13.2
- new net RS-12V: CN1.PWR, Q1.12V-IN, RS1.1
- new net RS-A: Q1.A, RS1.2
- new net RS-B: Q1.B, RS1.3
- new net SDA: I2C.2, U$1.P$3
- new net SLC: I2C.3, U$1.P$5
- net +5V: now also I2C.1
- net 10: now also R1.1, U$1.P$19; no longer R14.1
- net 11: now also U$1.P$23
- net 17: now also R10.1, R6.2, U$1.P$11; no longer R2.2, R3.1
- net 18: now also R5.2, R9.1, U$1.P$12; no longer R4.2, R8.1
- net 22: now also R2.2, R3.1, U$1.P$15; no longer R5.2, R9.1
- net 23: now also R11.1, R7.2, U$1.P$16; no longer R10.1, R6.2
- net 7: now also U$1.P$26
- net 8: now also U$1.P$24
- net 9: now also U$1.P$21
- net GND: now also I2C.4, RS1.4, U$2.P$1; no longer SL1.4, T1.E
- net N$15: now also T1.E, U$2.P$2; no longer R1.1
Routing:
- net 7: track 0.00 -> 89.7 mm, vias 0 -> 1
- net 8: track 0.00 -> 60.4 mm, vias 0 -> 1
- net 23: track 2.11 -> 39.9 mm
- net 25: track 0.00 -> 33.3 mm, vias 0 -> 1
- net N$19: track 30.1 -> 0.00 mm
- net 22: track 2.11 -> 31.2 mm
- net RS-12V: track 0.00 -> 27.2 mm
- net 10: track 0.00 -> 26.4 mm
- net 27: track 0.00 -> 24.8 mm
- net 11: track 0.00 -> 20.6 mm, vias 0 -> 1
- net +12V: track 79.9 -> 100.1 mm, vias 4 -> 3
- net 18: track 3.38 -> 22.8 mm
- net N$23: track 18.5 -> 0.00 mm
- net 24VAC-C: track 75.8 -> 58.4 mm
- net RS-A: track 0.00 -> 17.0 mm
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